File: PCB/03-ToF/03-ToF.brd (EAGLE design)
At the start: 80 x 80 mm, 84 parts, among them U2 PCA9555PW,112

Commit message: ねこ
Parts:
- moved R17 28.3 mm to (-19.4, -8.04), turned to 292.5 degrees
- moved R21 27.4 mm to (-8.04, 19.4), turned to 202.5 degrees
- moved R16 27.3 mm to (-14.8, -14.8), turned to 315 degrees
- moved R18 25.1 mm to (-21.0, 0.00)
- moved R19 22.3 mm to (-19.4, 8.04), turned to 247.5 degrees
- moved R20 19.5 mm to (-14.8, 14.8), turned to 225 degrees
- moved R6 18.8 mm to (0.00, 21.0), turned to 180 degrees
- moved R9 17.1 mm to (19.4, 8.04), turned to 112.5 degrees
- moved R15 16.8 mm to (-8.04, -19.4), turned to 337.5 degrees
- moved R7 15.6 mm to (8.04, 19.4), turned to 157.5 degrees
- moved R14 15.1 mm to (0.00, -21.0), turned to 0 degrees
- moved R10 13.7 mm to (21.0, 0.00)
- moved R13 13.4 mm to (8.04, -19.4), turned to 22.5 degrees
- moved R12 12.0 mm to (14.8, -14.8), turned to 45 degrees
- moved R8 12.0 mm to (14.8, 14.8), turned to 135 degrees
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
Commit message: おｋ
Routing:
- net GND: track 0.00 -> 564.0 mm, vias 0 -> 45
- net +3V3: track 0.00 -> 362.3 mm, vias 0 -> 6
- net +5V: track 0.00 -> 304.1 mm, vias 0 -> 6
- net SDA: track 0.00 -> 271.3 mm, vias 0 -> 10
- net SCL: track 0.00 -> 249.9 mm, vias 0 -> 5
- net X16: track 0.00 -> 59.7 mm
- net LED_SIG: track 0.00 -> 58.9 mm, vias 0 -> 6
- net VDD: track 0.00 -> 42.2 mm, vias 0 -> 4
- net X12: track 0.00 -> 40.8 mm, vias 0 -> 2
- net X11: track 0.00 -> 38.0 mm, vias 0 -> 1
- net X5: track 0.00 -> 33.4 mm
- net X14: track 0.00 -> 31.4 mm
- net X13: track 0.00 -> 29.8 mm
- net X15: track 0.00 -> 29.2 mm
- net X2: track 0.00 -> 26.1 mm, vias 0 -> 1
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- added copper zone on layer 1, net GND
- added copper zone on layer 16, net GND

Commit message: 03-tof
Parts:
- R3, R4: value 180 -> 1k
Routing:
- net GND: vias 45 -> 37
