File: PCB/03-ToF/03-ToF.sch (EAGLE design)
At the start: 84 parts, among them U2 PCA9555PW,112

Commit message: 03-tof
Parts:
- R3, R4: value 180 -> 1k
Other:
- moved on the sheet: C1, C2, C3, C4, D1, LED40, LED41, R1, R10, R11, R12, R13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
