File: PCB/01-main/002-main.sch (EAGLE design)
At the start: 84 parts, among them U2 PCA9555PW,112

Commit message: 電源基板完成
Parts:
- removed LED19, LED20, LED21, LED22, LED23, LED24, LED25, LED26, LED27, LED28, LED29, LED30, LED31, LED32: WS2812B_5050N, microbuilder:WS2812B_5050N
- removed LED40, LED41: BLUE, led:LEDSML0603
- removed TP1, TP3, TP4, TP5: PTR1TP10R, testpad:PTR1TP10R
- removed TP2: PTR1TP10SQ, testpad:PTR1TP10SQ
- removed VL1, VL10, VL11, VL12, VL13, VL14, VL15, VL16, VL2, VL3, VL4, VL5, VL6, VL7, VL8, VL9: VL53L0X, VL53L0X:VL53L0X
- added C10, C12, C13, C15, C9: 100μ, rcl:CPOL-EU153CLV-0505
- added C11, C14, C16, C5, C6, C7: 0.1µ, rcl:C-EUC0603
- added C8: 1µ, rcl:C-EUC0603
- added D2, D3: 1N4001, diode:GF1
- added IC1, IC2: NJU77551F, burr-brown:OPA340N
- added J1, J13, J2: 5267-4, con-molex-spox:5267-4
- added J10, J11, J12, J9: 22057045, con-molex-5268:22057045
- added J3, J4, J5, J6, J7: 22057035, con-molex-5268:22057035
- added J8: 5267-5, con-molex-spox:5267-5
- added JP1, JP2: JP2, jp:JP2
- added LS1: MLT-8530, MLT-8530:MLT-8530
- added Q1: C1015, transistor-pnp:BCX71SMD
- added R22, R23, R26, R27, R28, R29: 1k, rcl:R-EU_R0402
- added R24, R25: 330k, rcl:R-EU_R0402
- added R30, R31: 10k, rcl:R-EU_R0402
- added R32: 270, rcl:R-EU_R0402
- added REG2: REG-5V, #001-line:MYPARTS_NJM7800S-REGULATOR
- added S1: (no value), switch-omron:31-XX
- added SW1: SK-12D11VG3, Slide Switch:SK-12D11VG3
- added T1, T2, T3: BSS138, zetex:NMOSSOT23
- added U4: (no value), BNO055:BNO055
- added U5: MAX485ESA+T, MAX485:MAX485ESA+T
- added X1: Seeed Studio XIAO ESP32C3, Seeeduino XIAO:SEEEDUINO-XIAO-DIP
- added X2, X3: usb-c, microbuilder:USB_C
- added XT1: XT-30_L, XT-30:XT-30_L
- C1: value 0.1μ -> 4.7µ; device rcl:C-EUC0402 -> rcl:C-EUC0603
- C2: value 1μ -> 0.1µ; device rcl:C-EUC0402 -> rcl:C-EUC0603
- C3, C4: value 100μ -> 0.1µ; device rcl:CPOL-EU153CLV-0505 -> rcl:C-EUC0603
- D1: value 1N4007 -> 1N4001
- LED1, LED10, LED11, LED12, LED13, LED14, LED2, LED3, LED4, LED5, LED6, LED7, LED8, LED9: value WS2812B_5050N -> WS2812B_2020; device microbuilder:WS2812B_5050N -> microbuilder:WS2812B_2020
- LED15, LED16: value WS2812B_5050N -> BLUE; device microbuilder:WS2812B_5050N -> led:LEDSML0603
- LED17, LED18: value WS2812B_5050N -> WHITE; device microbuilder:WS2812B_5050N -> led:LEDSML0603
- R1, R2, R7, R8: value 10k -> 5k1
- R10, R9: value 10k -> 270
- R11: value 10k -> 180k
- R14: value 10k -> 20k
- R15, R16: value 10k -> 2k2
- R17: value 10k -> 7.5k
- R18, R19: value 10k -> 1k
- R20, R21: value 10k -> 330k
- R3: value 1k -> 270
- R4: value 1k -> 10k
- REG1: value NJM7805 -> REG-3V3
- U1: value (none) -> CH340ESMD; device Seeeduino XIAO:MOUDLE-SEEEDUINO-XIAO -> CH340E:CH340ESMD
- U2: value PCA9555PW,112 -> STM32F446RET6; device PCA9555PW_112:PCA9555PW,112 -> F446RE:STM32F446RET6
Connections:
- removed net LED_SIG: LED1.DI, TP5.TP
- removed net N$13 (its old number): LED14.DO, LED15.DI
- removed net N$33: LED18.DO, LED19.DI
- removed net N$34: LED27.DO, LED28.DI
- removed net N$7 (its old number): LED7.DO, LED8.DI
- removed net RX: TP3.TP, U1.PB09_A7_D7_RX
- removed net TX: TP4.TP, U1.PB08_A6_D6_TX
- removed net X1: R6.2, U2.IO0_2, VL1.XSHUT
- removed net X10: R15.2, U2.IO1_1, VL10.XSHUT
- removed net X11: R16.2, U2.IO0_4, VL11.XSHUT
- removed net X12: R17.2, U2.IO0_3, VL12.XSHUT
- removed net X13: R18.2, U2.IO0_5, VL13.XSHUT
- removed net X14: R19.2, U2.IO0_6, VL14.XSHUT
- removed net X15: R20.2, U2.IO0_7, VL15.XSHUT
- removed net X16: R21.2, U2.IO1_0, VL16.XSHUT
- removed net X2: R7.2, U2.IO0_1, VL2.XSHUT
- removed net X3: R8.2, U2.IO0_0, VL3.XSHUT
- removed net X4: R9.2, U2.IO1_7, VL4.XSHUT
- removed net X5: R10.2, U2.IO1_6, VL5.XSHUT
- removed net X6: R11.2, U2.IO1_5, VL6.XSHUT
- removed net X7: R12.2, U2.IO1_4, VL7.XSHUT
- removed net X8: R13.2, U2.IO1_3, VL8.XSHUT
- removed net X9: R14.2, U2.IO1_2, VL9.XSHUT
- new net !RE: Q1.C, R14.1, U5.!RE, U5.DE
- new net BOOT0: R31.1, SW1.P, U2A.BOOT0
- new net CTS: U1.CTS
- new net D+: U1.UD+, X2.D+, X3.D+
- new net D-: U1.UD-, X2.D-, X3.D-
- new net LCELL-L: IC1.OUT, R21.1
- new net LCELL-R: IC2.OUT, R25.1
- new net LED-FLOOR: J11.4, U2A.PB15
- new net LED-L: JP1.1, R27.2, T2.S, U2A.PA15
- new net LED-L-5V: JP1.2, LED1.DI, R26.2, T2.D
- new net LED-R: JP2.1, R29.2, T3.S, U2A.PB13
- new net LED-R-5V: JP2.2, LED8.DI, R28.2, T3.D
- new net LED-TOP: J8.-5, U2A.PC1
- new net LED-UI: J9.2, U2A.PB14
- new net LED-WHITE: LED17.A, U2A.PB12
- new net N$28: R15.2, R16.1, U5.B
- new net N$47: R7.1, X3.CC1
- new net N$48: R8.1, X3.CC2
- new net N$49: LED15.A, X2.VBUS
- new net N$50: LED16.A, X3.VBUS
- new net N$51: LED16.C, R9.2
- new net N$8: C14.1, U1.V3
- new net NRST: C16.1, J13.-3, R30.2, S1.P, U2A.NRST
- new net RTS: U1.RTS
- new net SERVO-SIG: J3.1, J4.1, J5.1, J6.1, J7.1, U5.A
- new net SIG-FLOOR: J11.3, R11.2, U2A.PC0
- new net SPK: T1.G, U2A.PB6
- new net SW1: J9.4, R5.2, U2A.PA4
- new net SW2: J9.3, R6.2, U2A.PA5
- new net SWCLK: J13.-1, U2A.PA14
- new net SWDIO: J13.-2, U2A.PA13
- new net SWO: U2A.PB3
- new net TOGGLE: J9.1, R4.2, U2A.PA6
- new net UART1-RX: U1.TX, U2A.PA10
- new net UART1-TX: U1.RX, U2A.PA9
- new net UART2-RX: J2.-4, U2A.PA3
- new net UART2-TX: J2.-3, U2A.PA2
- new net UART3-RX: U2A.PC5, X1.PB08_A6_D6_TX
- new net UART3-TX: U2A.PB10, X1.PB09_A7_D7_RX
- new net UART4-RX: J8.-4, U2A.PA1
- new net UART4-TX: J8.-3, U2A.PA0
- new net UART5-RX: U2A.PD2, U5.RO
- new net UART5-TX: R17.2, U2A.PC12, U5.DI
- new net UART6-RX: J1.-4, U2A.PC7
- new net UART6-TX: J1.-3, U2A.PC6
- net +3V3: now also C2.1, C3.1, C4.1, C5.1, C6.1, C7.1, D1.A, IC1.V+, IC2.V+, J10.1, J12.1, LS1.1, R27.1, R29.1, R30.1, R4.1, R5.1, REG1.VOUT, SW1.O, T2.G, T3.G, U2B.VBAT, U2B.VDD, U2B.VDDA/VREF+, U2B.VDD_2, U2B.VDD_3, U2B.VDD_4, U4.VIN; no longer LED41.A, R1.2, R10.1, R11.1, R14.1, R15.1, R16.1, R17.1, R18.1, R19.1, R2.2, R20.1, R21.1, R5.2, R7.1, R8.1, R9.1, U1.3V3, U2.VDD, VL1.VCC, VL10.VCC, VL11.VCC, VL12.VCC, VL13.VCC, VL14.VCC, VL15.VCC, VL16.VCC, VL2.VCC, VL3.VCC, VL4.VCC, VL5.VCC, VL6.VCC, VL7.VCC, VL8.VCC, VL9.VCC
- net +5V: now also C11.1, D2.A, D3.A, J1.-2, J11.1, J2.-2, Q1.E, R11.1, R15.1, R26.1, R28.1, REG2.VOUT, U1.VCC, U5.VCC; no longer C1.1, C3.+, D1.A, LED15.VDD, LED16.VDD, LED17.VDD, LED18.VDD, LED19.VDD, LED20.VDD, LED21.VDD, LED22.VDD, LED23.VDD, LED24.VDD, LED25.VDD, LED26.VDD, LED27.VDD, LED28.VDD, LED29.VDD, LED30.VDD, LED31.VDD, LED32.VDD, LED40.A, REG1.VOUT, U1.5V
- net GND: now also C10.-, C11.2, C12.-, C13.-, C14.2, C15.-, C16.2, C3.2, C4.2, C5.2, C6.2, C7.2, C8.2, C9.-, IC1.V-, IC2.V-, J1.-1, J10.2, J11.2, J12.2, J13.-4, J2.-1, J3.2, J4.2, J5.2, J6.2, J7.2, J8.-2, LED18.C, R1.2, R14.2, R16.2, R2.2, R20.1, R24.1, R3.1, R31.2, R32.1, R7.2, R8.2, R9.1, REG2.GND, S1.S, SW1.CASE, T1.S, U2B.VSS, U2B.VSSA/VREF-, U2B.VSS_2, U2B.VSS_3, U2B.VSS_4, U4.GND, U5.GND, X1.GND, X2.GND, X3.GND, XT1.2; no longer C3.-, C4.-, LED15.GND, LED16.GND, LED17.GND, LED18.GND, LED19.GND, LED20.GND, LED21.GND, LED22.GND, LED23.GND, LED24.GND, LED25.GND, LED26.GND, LED27.GND, LED28.GND, LED29.GND, LED30.GND, LED31.GND, LED32.GND, R3.2, R4.2, TP2.TP, U2.A0, U2.A1, U2.A2, U2.VSS, VL1.GND, VL10.GND, VL11.GND, VL12.GND, VL13.GND, VL14.GND, VL15.GND, VL16.GND, VL2.GND, VL3.GND, VL4.GND, VL5.GND, VL6.GND, VL7.GND, VL8.GND, VL9.GND
- net N$14: now also R1.1, X2.CC1; no longer LED15.DO, LED16.DI
- net N$15: now also R2.1, X2.CC2; no longer LED16.DO, LED17.DI
- net N$16: now also LED15.C, R3.2; no longer LED17.DO, LED18.DI
- net N$17: now also LS1.2, T1.D; no longer LED19.DO, LED20.DI
- net N$18: now also C1.1, U2B.VCAP_1; no longer LED20.DO, LED21.DI
- net N$19: now also IC1.+IN, R18.1, R20.2; no longer LED21.DO, LED22.DI
- net N$20: now also IC1.-IN, R19.1, R21.2; no longer LED22.DO, LED23.DI
- net N$21: now also J10.3, R19.2; no longer LED23.DO, LED24.DI
- net N$22: now also R10.2, U1.TNOW; no longer LED24.DO, LED25.DI
- net N$23: now also LED18.A, R10.1; no longer LED40.C, R3.1
- net N$24: now also J10.4, R18.2; no longer LED41.C, R4.1
- net N$25: now also IC2.+IN, R22.1, R24.2; no longer R5.1, U2.!INT
- net N$26: now also IC2.-IN, R23.1, R25.2; no longer LED25.DO, LED26.DI
- net N$27: now also Q1.B, R17.1; no longer LED26.DO, LED27.DI
- net N$29: now also J12.4, R22.2; no longer LED28.DO, LED29.DI
- net N$30: now also J12.3, R23.2; no longer LED29.DO, LED30.DI
- net N$31: now also D3.C, X1.5V; no longer LED30.DO, LED31.DI
- net N$32: now also LED17.C, R32.2; no longer LED31.DO, LED32.DI
- net SCL: now also R13.2, U2A.PB8, U4.SCL; no longer R2.1, U1.PA9_A5_D5_SCL, U2.SCL, VL1.SCL, VL10.SCL, VL11.SCL, VL12.SCL, VL13.SCL, VL14.SCL, VL15.SCL, VL16.SCL, VL2.SCL, VL3.SCL, VL4.SCL, VL5.SCL, VL6.SCL, VL7.SCL, VL8.SCL, VL9.SCL
- net SDA: now also R12.2, U2A.PB9, U4.SDA; no longer R1.1, U1.PA8_A4_D4_SDA, U2.SDA, VL1.SDA, VL10.SDA, VL11.SDA, VL12.SDA, VL13.SDA, VL14.SDA, VL15.SDA, VL16.SDA, VL2.SDA, VL3.SDA, VL4.SDA, VL5.SDA, VL6.SDA, VL7.SDA, VL8.SDA, VL9.SDA
- net VDD: now also C10.+, C12.+, C13.+, C15.+, C8.1, C9.+, D2.C, J3.3, J4.3, J5.3, J6.3, J7.3, J8.-1, REG2.VIN, XT1.1; no longer C2.1, C4.+, TP1.TP
Other:
- note added: "BNO055"
- note added: "BOOT0"
- note added: "CAM"
- note added: "CH340E"
- note added: "CONN-SERVO"
- note added: "DEBUG"
- note added: "FLOOR"
- note added: "LOAD CELL"
- note added: "Logic Level Converter"
- note added: "NEOPIXEL"
- note added: "Pull-up"
- note added: "REG"
- note added: "RESET"
- note added: "RS485"
- note added: "SPK"
- note added: "STM32F446RE"
- note added: "TOP"
- note added: "UI"
- note added: "USB-C"
- note added: "XT30"
- note removed: "CONN"
- note removed: "PCA9555"
- note removed: "PULL UP"
- note removed: "REGULATOR"
- note removed: "VL53L0X"
