File: PCB/01-main/01-main.sch (EAGLE design)
At the start: 76 parts, among them CN1 ML8, J1 22057045, J14 22057055, J8 22057045, Q1 C1015, SW1 SK-12D11VG3, T1 BSS138, U1 CH340ESMD, U2 STM32F446RET6, U5 MAX485ESA+T, X1 Seeed Studio XIAO ESP32C3, X2 usb-c

Commit message: 配置完了
Connections:
- removed net SW1: U2A.PA4
- removed net SW2: U2A.PA5
Changed lines of the file:
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@@
 <setting verticaltext="up"/>
 </settings>
-<grid distance="0.1" unitdist="inch" unit="inch" style="lines" multiple="1" display="yes" altdistance="0.01" altunitdist="inch" altunit="inch"/>
+<grid distance="0.1" unitdist="inch" unit="inch" style="lines" multiple="1" display="no" altdistance="0.01" altunitdist="inch" altunit="inch"/>
 <layers>
 <layer number="1" name="Top" color="4" fill="1" visible="no" active="no"/>
@@
 </segment>
 </net>
-<net name="SW1" class="0">
-<segment>
-<pinref part="U2" gate="A" pin="PA4"/>
-<wire x1="124.46" y1="116.84" x2="116.84" y2="116.84" width="0.1524" layer="91"/>
-<label x="104.14" y="116.84" size="1.778" layer="95"/>
-</segment>
-</net>
-<net name="SW2" class="0">
-<segment>
-<pinref part="U2" gate="A" pin="PA5"/>
-<wire x1="124.46" y1="114.3" x2="116.84" y2="114.3" width="0.1524" layer="91"/>
-<label x="104.14" y="114.3" size="1.778" layer="95"/>
-</segment>
-</net>

Commit message: メイン配置おわ
Parts:
- removed C10, C12, C15: 100μ, rcl:CPOL-EU153CLV-0505
- removed D3: 1N4001, diode:GF1
- removed X1: Seeed Studio XIAO ESP32C3, Seeeduino XIAO:SEEEDUINO-XIAO-DIP
- added U3: SUNA_LIB_M5STAMP_C3U_MATE, M5StampC3-pin:SUNA_LIB_M5STAMP_C3U_MATE
Connections:
- removed net N$31: D3.C, X1.5V
- net +5V: now also U3.5V1, U3.5V2; no longer D3.A
- net GND: now also U3.GND2, U3.GND3, U3.GND4; no longer C10.-, C12.-, C15.-, X1.GND
- net UART3-TX: now also U3.G20; no longer X1.PB09_A7_D7_RX
- net VDD: no longer C10.+, C12.+, C15.+
Other:
- moved on the sheet: C13
