File: PCB/01-main/01-main.brd (EAGLE design)
At the start: 106 x 53 mm, 72 parts, among them CN1 ML8, J1 22057045, J14 22057055, J8 22057045, Q1 C1015, SW1 SK-12D11VG3, T1 BSS138, U1 CH340ESMD, U2 STM32F446RET6, U3 SUNA_LIB_M5STAMP_C3U_MATE, U5 MAX485ESA+T, X2 usb-c

Commit message: wei
Routing:
- net VDD: track 73.3 -> 89.6 mm, vias 2 -> 3
Changed lines of the file:
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@@
 <wire x1="-38" y1="15" x2="-46" y2="15" width="0.508" layer="16"/>
 <via x="-38" y="15" extent="1-16" drill="0.35"/>
-<wire x1="5" y1="6.5" x2="1.95" y2="12" width="0" layer="19" extent="1-1"/>
-<wire x1="-4.85" y1="14" x2="1.72" y2="14.2" width="0" layer="19" extent="1-1"/>
+<wire x1="-3.113025" y1="10.515" x2="-0.786975" y2="10.515" width="1.016" layer="1"/>
+<wire x1="-6.05" y1="12" x2="-4.598025" y2="12" width="1.016" layer="1"/>
+<wire x1="0.698025" y1="12" x2="1.95" y2="12" width="1.016" layer="1"/>
+<wire x1="-3.113025" y1="10.515" x2="-4.598025" y2="12" width="1.016" layer="1"/>
+<wire x1="-0.1509875" y1="11.1509875" x2="0.698025" y2="12" width="1.016" layer="1"/>
+<via x="-0.1509875" y="11.1509875" extent="1-16" drill="0.35"/>
+<wire x1="-0.786975" y1="10.515" x2="-0.1509875" y2="11.1509875" width="1.016" layer="1"/>
+<wire x1="-0.1509875" y1="11.1509875" x2="0.3490125" y2="11.1509875" width="1.016" layer="16"/>
+<wire x1="0.3490125" y1="11.1509875" x2="5" y2="6.5" width="1.016" layer="16"/>
 </signal>
 <signal name="SERVO-SIG">

Commit message: cat
Routing:
- net +3V3: track 2.30 -> 18.2 mm
- net GND: track 322.7 -> 337.0 mm
- net NRST: track 0.00 -> 3.88 mm
- net N$18: track 0.00 -> 2.18 mm
- net TOGGLE: track 0.00 -> 1.97 mm

Commit message: ねこ
Routing:
- net +5V: track 27.1 -> 262.2 mm, vias 0 -> 3
- net GND: track 337.0 -> 545.5 mm, vias 21 -> 124
- net +3V3: track 18.2 -> 222.0 mm, vias 0 -> 9
- net LOADCELL-L: track 0.00 -> 104.1 mm, vias 0 -> 2
- net SIG-FLOOR: track 0.00 -> 93.9 mm, vias 0 -> 3
- net LED-R: track 0.00 -> 87.0 mm, vias 0 -> 4
- net UART6-TX: track 0.00 -> 84.2 mm, vias 0 -> 2
- net LED-L: track 0.00 -> 78.9 mm, vias 0 -> 4
- net TOGGLE: track 1.97 -> 60.9 mm, vias 0 -> 3
- net SPK: track 0.00 -> 55.6 mm, vias 0 -> 2
- net UART6-RX: track 0.00 -> 53.9 mm, vias 0 -> 2
- net LOADCELL-R: track 0.00 -> 51.2 mm, vias 0 -> 5
- net LED-WHITE: track 0.00 -> 48.8 mm, vias 0 -> 2
- net LED-TOP: track 0.00 -> 39.9 mm, vias 0 -> 3
- net NRST: track 3.88 -> 42.0 mm, vias 0 -> 1
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- added copper zone on layer 1, net GND
- added copper zone on layer 16, net GND
