File: PCB/02-UI/02-ui.sch (EAGLE design)
At the start: 15 parts, among them X1 SEEEDUINO-XIAO-DIP

Commit message: 02-ui
Parts:
- added JP1: (no value), pinhead-compact:PINHD-1X2
- added Q2: BSS84, transistor-small-signal:BSS84
- added TFT1: 2.8TFT, 2.8TFT:2.8TFT
- added TP1: TPTP10SQ, testpad:TPTP10SQ
- added TP2, TP3, TP4, TP5, TP6: TPTP10R, testpad:TPTP10R
Connections:
- removed net NEOPIXEL: LED1.DI
- new net +3V3: Q2.S, TFT1.VCC, X1.3V3
- new net BACKLIGHT: Q2.G, X1.PA11_A3_D3
- new net BIN: JP1.2, TP5.TP
- new net LED: LED1.DI, TP6.TP
- new net MISO: TFT1.T_DO, X1.PA5_A9_D9_MISO
- new net MOSI: TFT1.MOSI, TFT1.T_DIN, X1.PA6_A10_D10_MOSI
- new net RX: TP3.TP, X1.PB09_A7_D7_RX
- new net SCK: TFT1.SCK, TFT1.T_CLK, X1.PA7_A8_D8_SCK
- new net TFT_CS: TFT1.CS, X1.PA02_A0_D0
- new net TFT_DC: TFT1.DC, X1.PA10_A2_D2
- new net TFT_LED: Q2.D, TFT1.LED
- new net TFT_RST: TFT1.RST, X1.PA4_A1_D1
- new net TOUCH_CS: TFT1.T_CS, X1.PA9_A5_D5_SCL
- new net TOUCH_IRQ: TFT1.T_IRQ, X1.PA8_A4_D4_SDA
- new net TX: TP4.TP, X1.PB08_A6_D6_TX
- net +5V: now also TP2.TP, X1.5V
- net GND: now also JP1.1, TFT1.GND, TP1.TP, X1.GND
Other:
- note added: "CONN"
- note added: "NEOPIXEL"
- note added: "TOGGLE"
- note added: "XIAO RP2040"
