File: PCB/02-UI/02-ui.brd (EAGLE design)
At the start: 105 x 60 mm, 24 parts, among them Q2 BSS84, X1 SEEEDUINO-XIAO-DIP

Commit message: 微調整
Parts:
- moved TP2 1.27 mm to (44.5, -20.3)
- moved TP3 1.27 mm to (43.2, -20.3)
- moved TP5 1.27 mm to (40.6, -20.3)
- moved TP1 1.27 mm to (45.7, -20.3)
- moved TP4 1.27 mm to (41.9, -20.3)
- moved TP6 1.27 mm to (39.4, -20.3)
Routing:
- net RX: track 28.1 -> 29.3 mm
- net TX: track 9.09 -> 10.4 mm
- net LED: track 57.0 -> 58.3 mm
- net +5V: track 124.1 -> 123.4 mm
Other:
- outline, holes or cut-outs redrawn

Commit message: main配置完了
Parts:
- moved JP1 0.50 mm to (43.5, -46.0)
Other:
- outline, holes or cut-outs redrawn
Changed lines of the file:
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@@
 <drawing>
 <settings>
-<setting alwaysvectorfont="yes"/>
+<setting alwaysvectorfont="no"/>
 <setting verticaltext="up"/>
 </settings>
-<grid distance="50" unitdist="mil" unit="mil" style="lines" multiple="1" display="yes" altdistance="10" altunitdist="mil" altunit="mil"/>
+<grid distance="1" unitdist="mm" unit="mm" style="lines" multiple="1" display="yes" altdistance="0.5" altunitdist="mm" altunit="mm"/>
 <layers>
 <layer number="1" name="Top" color="4" fill="1" visible="yes" active="yes"/>
@@
 <wire x1="-52.5" y1="-62.619240625" x2="-51.914209375" y2="-64.03345" width="0.05" layer="20" curve="45"/>
 <rectangle x1="-53" y1="-68.961" x2="-47.498" y2="-12" layer="42"/>
-<circle x="43" y="-54" radius="4" width="0.1524" layer="42"/>
-<rectangle x1="40" y1="-58.5" x2="46" y2="-49.5" layer="26"/>
+<circle x="43.5" y="-54" radius="4" width="0.1524" layer="42"/>
+<rectangle x1="40.5" y1="-58.5" x2="46.5" y2="-49.5" layer="26"/>
 <circle x="-30" y="-70.447659375" radius="1.05" width="0.05" layer="20"/>
 <circle x="30" y="-70.447659375" radius="1.05" width="0.05" layer="20"/>
@@
 <rectangle x1="47.5" y1="-21" x2="52.5" y2="-12.5" layer="42"/>
 <rectangle x1="47.5" y1="-68.5" x2="52.5" y2="-39" layer="42"/>
-<circle x="43" y="-54" radius="2.6" width="0.1524" layer="20"/>
-<circle x="43" y="-54" radius="4" width="0.1524" layer="41"/>
+<circle x="43.5" y="-54" radius="2.6" width="0.1524" layer="20"/>
+<circle x="43.5" y="-54" radius="4" width="0.1524" layer="41"/>
 <rectangle x1="13.11" y1="-70.81" x2="13.57" y2="-70.79" layer="26" rot="R180"/>
 <rectangle x1="-11.53" y1="-70.81" x2="-11.33" y2="-70.79" layer="26" rot="R180"/>
@@
 <attribute name="TP_SIGNAL_NAME" value="" x="39.37" y="-22.225" size="1" layer="38" rot="MR0"/>
 </element>
-<element name="JP1" library="pinhead-compact" package="1X02" package3d_urn="urn:adsk.eagle:package:22435/2" value="" x="43" y="-46" smashed="yes" rot="MR180">
-<attribute name="POPULARITY" value="98" x="43" y="-46" size="1.778" layer="28" rot="MR180" display="off"/>
-<attribute name="VALUE" x="40.46" y="-42.825" size="1.27" layer="28" rot="MR180"/>
+<element name="JP1" library="pinhead-compact" package="1X02" package3d_urn="urn:adsk.eagle:package:22435/2" value="" x="43.5" y="-46" smashed="yes" rot="MR180">
+<attribute name="POPULARITY" value="98" x="43.5" y="-46" size="1.778" layer="28" rot="MR180" display="off"/>
+<attribute name="VALUE" x="40.96" y="-42.825" size="1.27" layer="28" rot="MR180"/>
 </element>
 <element name="Q2" library="transistor-small-signal" library_urn="urn:adsk.eagle:library:401" package="SOT23" package3d_urn="urn:adsk.eagle:package:28738/2" value="BSS84" x="42" y="-29" smashed="yes">
@@
 <wire x1="45.72" y1="-23.967175" x2="44.4881" y2="-22.735275" width="0.381" layer="16"/>
 <wire x1="44.4881" y1="-22.735275" x2="44.4881" y2="-21.5519" width="0.381" layer="16"/>
-<wire x1="41.73" y1="-49.23596875" x2="41.73" y2="-46" width="0.381" layer="16"/>
-<wire x1="38.7333" y1="-52.23266875" x2="41.73" y2="-49.23596875" width="0.381" layer="16"/>
-<wire x1="41.73" y1="-46" x2="45.72" y2="-42.01" width="0.381" layer="1"/>
-<wire x1="45.72" y1="-42.01" x2="45.72" y2="-37.465" width="0.381" layer="1"/>
+<wire x1="42.23" y1="-48.73596875" x2="42.23" y2="-46" width="0.381" layer="16"/>
+<wire x1="38.7333" y1="-52.23266875" x2="42.23" y2="-48.73596875" width="0.381" layer="16"/>
+<wire x1="42.23" y1="-46" x2="45.72" y2="-42.51" width="0.381" layer="1"/>
+<wire x1="45.72" y1="-42.51" x2="45.72" y2="-37.465" width="0.381" layer="1"/>
 <wire x1="28.5345" y1="-69.840625" x2="29.39296875" y2="-68.98215625" width="0.381" layer="1"/>
 <wire x1="27.3815125" y1="-71.7175" x2="28.5345" y2="-70.5645125" width="0.381" layer="1"/>
@@
 <wire x1="-22.4184875" y1="-69.2825" x2="-24.0019125" y2="-69.2825" width="0.381" layer="1"/>
 <wire x1="-24.0019125" y1="-69.2825" x2="-24.6694125" y2="-69.95" width="0.381" layer="1"/>
-<wire x1="38.7333" y1="-52.23266875" x2="41.23266875" y2="-49.7333" width="0.381" layer="1"/>
-<wire x1="41.23266875" y1="-49.7333" x2="42.278875" y2="-49.7333" width="0.381" layer="1"/>
-<wire x1="42.278875" y1="-49.7333" x2="48.26" y2="-43.752175" width="0.381" layer="1"/>
-<wire x1="48.26" y1="-43.752175" x2="48.26" y2="-37.465" width="0.381" layer="1"/>
 <wire x1="36.50569375" y1="-53.6275" x2="37.40930625" y2="-53.6275" width="0.381" layer="1"/>
-<wire x1="37.40930625" y1="-53.6275" x2="38.7333" y2="-52.30350625" width="0.381" layer="1"/>
-<wire x1="38.7333" y1="-52.30350625" x2="38.7333" y2="-52.23266875" width="0.381" layer="1"/>
 <wire x1="35.2845" y1="-54.84869375" x2="36.50569375" y2="-53.6275" width="0.381" layer="1"/>
-<wire x1="35.2845" y1="-62.5853" x2="35.2845" y2="-54.84869375" width="0.381" layer="1"/>
 <wire x1="48.26" y1="-24.5028125" x2="48.26" y2="-37.465" width="0.381" layer="16"/>
 <wire x1="47.0281" y1="-23.2709125" x2="48.26" y2="-24.5028125" width="0.381" layer="16"/>
-<wire x1="32.9408" y1="-64.929" x2="35.2845" y2="-62.5853" width="0.381" layer="1"/>
-<wire x1="26.9" y1="-69.95" x2="31.921" y2="-64.929" width="0.381" layer="1"/>
-<wire x1="31.921" y1="-64.929" x2="32.9408" y2="-64.929" width="0.381" layer="1"/>
 <wire x1="44.45" y1="-20.32" x2="44.45" y2="-20.1409875" width="0.381" layer="16"/>
 <wire x1="44.45" y1="-20.1409875" x2="45.0884875" y2="-19.5025" width="0.381" layer="16"/>
@@
 <wire x1="46.3515125" y1="-19.5025" x2="47.0281" y2="-20.1790875" width="0.381" layer="16"/>
 <wire x1="47.0281" y1="-20.1790875" x2="47.0281" y2="-23.2709125" width="0.381" layer="16"/>
+<wire x1="35.2845" y1="-61.5655" x2="35.2845" y2="-54.84869375" width="0.381" layer="1"/>
+<wire x1="41.30350625" y1="-49.7333" x2="42.778875" y2="-49.7333" width="0.381" layer="1"/>
+<wire x1="42.778875" y1="-49.7333" x2="48.26" y2="-44.252175" width="0.381" layer="1"/>
+<wire x1="48.26" y1="-44.252175" x2="48.26" y2="-37.465" width="0.381" layer="1"/>
+<wire x1="26.9" y1="-69.95" x2="35.2845" y2="-61.5655" width="0.381" layer="1"/>
+<wire x1="37.40930625" y1="-53.6275" x2="41.30350625" y2="-49.7333" width="0.381" layer="1"/>
 </signal>
 <signal name="N$9">
@@
 <contactref element="TP5" pad="TP"/>
 <contactref element="JP1" pad="2"/>
-<wire x1="44.27" y1="-46" x2="44.27" y2="-38.117175" width="0.381" layer="16"/>
-<wire x1="44.27" y1="-38.117175" x2="44.4119" y2="-37.975275" width="0.381" layer="16"/>
-<wire x1="44.4119" y1="-37.975275" x2="44.4119" y2="-36.4119" width="0.381" layer="16"/>
-<wire x1="44.4119" y1="-36.4119" x2="40.83" y2="-32.83" width="0.381" layer="16"/>
-<wire x1="40.83" y1="-32.83" x2="40.64" y2="-32.64" width="0.381" layer="16"/>
+<wire x1="44.4119" y1="-36.4119" x2="44.4119" y2="-45.6419" width="0.381" layer="16"/>
+<wire x1="44.77" y1="-46" x2="44.4119" y2="-45.6419" width="0.381" layer="16"/>
+<wire x1="44.4119" y1="-36.4119" x2="39.4081" y2="-31.4081" width="0.381" layer="16"/>
 <wire x1="40.64" y1="-20.482825" x2="40.64" y2="-20.32" width="0.381" layer="16"/>
 <wire x1="39.4081" y1="-21.714725" x2="40.64" y2="-20.482825" width="0.381" layer="16"/>
-<wire x1="40.64" y1="-32.64" x2="39.4081" y2="-31.4081" width="0.381" layer="16"/>
 <wire x1="39.4081" y1="-31.4081" x2="39.4081" y2="-21.714725" width="0.381" layer="16"/>
 </signal>
