File: PCB/04-bottom/04-bottom.brd (EAGLE design)
At the start: 128 x 128.5 mm, 7 parts

Commit message: 配置完了
Parts:
- added AMP1, AMP2: NJU77551F, NJU77551F:SOT23-5
- added CN1: ML8-R, ML8:ML6
- added J1, J2, J3, J4, J7: 5267-3, con-molex-spox:5267-3
- added J5, J6: 22057045, con-molex-5268:CON_22057045_MOL
- added JP2, JP4: (no value), pinhead:1X02
- added JP3: (no value), pinhead:1X04
- added R1, R2, R5, R6: 1k, rcl:R0805
- added R3, R4, R7, R8: 330k, rcl:R0805
- moved U1 1.00 mm to (8.89, -38.4)
- moved JP1 0.59 mm to (-41.9, -63.2)
Connections:
- new net +3V3: AMP1.5, AMP2.5, J5.1, J6.1, JP1.1, JP3.1, U1.12
- new net LED-FLOOR: CN1.6
- new net LOADCELL-L: AMP1.4, CN1.4, R4.2
- new net LOADCELL-R: AMP2.4, CN1.3, R8.2
- new net MIRROR: CN1.8, U1.7
- new net N$1: J5.3, R2.1
- new net N$2: J5.4, R1.1
- new net N$3: AMP1.3, R2.2, R4.1
- new net N$4: AMP1.1, R1.2, R3.1
- new net N$5: J6.3, R6.1
- new net N$6: J6.4, R5.1
- new net N$7: AMP2.3, R6.2, R8.1
- new net N$8: AMP2.1, R5.2, R7.1
- new net SCL: JP1.3, JP3.3, U1.6
- new net SDA: JP1.4, JP3.4, U1.5
- new net SERVO-SIG: CN1.7, J1.P$1, J2.P$1, J3.P$1, J4.P$1, J7.P$1
- new net SIG-FLOOR: CN1.5
- new net VDD: CN1.2, J1.P$2, J2.P$2, J3.P$2, J4.P$2, J7.P$2, U1.14, VDD1.P$1
- new net XSHUT1: JP2.1, U1.11
- new net XSHUT2: JP4.1, U1.1
- net GND: now also AMP1.2, AMP2.2, CN1.1, J1.P$3, J2.P$3, J3.P$3, J4.P$3, J5.2, J6.2, J7.P$3, JP1.2, JP3.2, R3.2, R7.2, U1.13
Routing:
- net SERVO-SIG: track 0.00 -> 234.3 mm
- net VDD: track 0.00 -> 234.2 mm
- net GND: track 0.00 -> 206.7 mm
Other:
- board size 128 x 128.5 mm -> 128 x 129.5 mm

Commit message: にゅーぷるあっぷ
Parts:
- added R10, R9: 10k, rcl:R0402
- moved J5 1.00 mm to (22.5, -41.0)
- moved J6 1.00 mm to (-15.0, -41.0)
Connections:
- net +3V3: now also R10.2, R9.2
- net SCL: now also R10.1
- net SDA: now also R9.1

Commit message: 今度こそ配置完了？
Parts:
- added TP1, TP3, TP4: PTR1TP10R, testpad:TP10R
- added TP2: PTR1TP10SQ, testpad:TP10SQ
Connections:
- net +3V3: now also TP1.TP
- net GND: now also TP2.TP
- net LED-FLOOR: now also TP4.TP
- net SIG-FLOOR: now also TP3.TP
Other:
- outline, holes or cut-outs redrawn
Changed lines of the file:
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@@
 <drawing>
 <settings>
-<setting alwaysvectorfont="no"/>
+<setting alwaysvectorfont="yes"/>
 <setting verticaltext="up"/>
 </settings>
-<grid distance="1" unitdist="mm" unit="mm" style="lines" multiple="1" display="yes" altdistance="0.5" altunitdist="mm" altunit="mm"/>
+<grid distance="50" unitdist="mil" unit="mil" style="lines" multiple="1" display="yes" altdistance="25" altunitdist="mil" altunit="mil"/>
 <layers>
 <layer number="1" name="Top" color="4" fill="1" visible="yes" active="yes"/>
@@
 <circle x="-8.195" y="3.5" radius="2" width="0.05" layer="41"/>
 <circle x="-35" y="-60.5" radius="1" width="0.3" layer="100"/>
+<wire x1="35.56" y1="-66.04" x2="39.37" y2="-66.04" width="0.05" layer="20"/>
+<wire x1="39.37" y1="-66.04" x2="39.37" y2="-67.31" width="0.05" layer="20" curve="-180"/>
+<wire x1="35.56" y1="-67.31" x2="35.56" y2="-66.04" width="0.05" layer="20" curve="-180"/>
+<wire x1="39.37" y1="-67.31" x2="35.56" y2="-67.31" width="0.05" layer="20"/>
 </plain>
 <attributes>
@@
 <attribute name="POPULARITY" value="0" x="11" y="-44" size="1.778" layer="27" rot="R90" display="off"/>
 <attribute name="SPICEPREFIX" value="R" x="11" y="-44" size="1.778" layer="27" rot="R90" display="off"/>
+</element>
+<element name="TP1" library="testpad" library_urn="urn:adsk.eagle:library:385" package="TP10R" package3d_urn="urn:adsk.eagle:package:27959/1" value="PTR1TP10R" x="39.37" y="-64.77" smashed="yes">
+<attribute name="POPULARITY" value="0" x="39.37" y="-64.77" size="1.778" layer="27" display="off"/>
+<attribute name="TP_SIGNAL_NAME" value="" x="39.37" y="-64.77" size="1.778" layer="27" display="off"/>
+</element>
+<element name="TP2" library="testpad" library_urn="urn:adsk.eagle:library:385" package="TP10SQ" package3d_urn="urn:adsk.eagle:package:27962/1" value="PTR1TP10SQ" x="38.1" y="-64.77" smashed="yes">
+<attribute name="POPULARITY" value="0" x="38.1" y="-64.77" size="1.778" layer="27" display="off"/>
+<attribute name="TP_SIGNAL_NAME" value="" x="38.1" y="-64.77" size="1.778" layer="27" display="off"/>
+</element>
+<element name="TP3" library="testpad" library_urn="urn:adsk.eagle:library:385" package="TP10R" package3d_urn="urn:adsk.eagle:package:27959/1" value="PTR1TP10R" x="36.83" y="-64.77" smashed="yes">
+<attribute name="POPULARITY" value="0" x="36.83" y="-64.77" size="1.778" layer="27" display="off"/>
+<attribute name="TP_SIGNAL_NAME" value="" x="36.83" y="-64.77" size="1.778" layer="27" display="off"/>
+</element>
+<element name="TP4" library="testpad" library_urn="urn:adsk.eagle:library:385" package="TP10R" package3d_urn="urn:adsk.eagle:package:27959/1" value="PTR1TP10R" x="35.56" y="-64.77" smashed="yes">
+<attribute name="POPULARITY" value="0" x="35.56" y="-64.77" size="1.778" layer="27" display="off"/>
+<attribute name="TP_SIGNAL_NAME" value="" x="35.56" y="-64.77" size="1.778" layer="27" display="off"/>
 </element>
 </elements>
@@
 <wire x1="-13.66613125" y1="1.482" x2="-12" y2="-0.18413125" width="1.27" layer="16"/>
 <wire x1="-12" y1="-0.18413125" x2="-12" y2="-7.695" width="1.27" layer="16"/>
+<contactref element="TP2" pad="TP"/>
+<wire x1="-41.94" y1="-64.445" x2="38.1" y2="-64.77" width="0" layer="19" extent="1-1"/>
 <wire x1="-28.5" y1="-38.694" x2="-41.94" y2="-64.445" width="0" layer="19" extent="1-1"/>
 <wire x1="-29.45" y1="-36" x2="-28.5" y2="-38.694" width="0" layer="19" extent="1-1"/>
@@
 <wire x1="-8.11" y1="-53.95" x2="-17.4892" y2="-41" width="0" layer="19" extent="1-1"/>
 <wire x1="-49.5" y1="-16" x2="-29.45" y2="-36" width="0" layer="19" extent="1-1"/>
+<wire x1="25" y1="4" x2="25" y2="4" width="0" layer="19" extent="1-16"/>
+<wire x1="24" y1="3" x2="25" y2="4" width="0" layer="19" extent="16-16"/>
+<wire x1="26" y1="6" x2="25" y2="4" width="0" layer="19" extent="16-16"/>
+<wire x1="24" y1="6" x2="26" y2="6" width="0" layer="19" extent="1-1"/>
+<wire x1="27" y1="3" x2="25" y2="4" width="0" layer="19" extent="16-16"/>
+<wire x1="30" y1="3" x2="27" y2="3" width="0" layer="19" extent="1-1"/>
+<wire x1="30" y1="6" x2="30" y2="3" width="0" layer="19" extent="1-1"/>
+<wire x1="33" y1="3" x2="30" y2="3" width="0" layer="19" extent="1-1"/>
+<wire x1="36" y1="3" x2="33" y2="3" width="0" layer="19" extent="1-1"/>
+<wire x1="29" y1="9" x2="30" y2="6" width="0" layer="19" extent="1-1"/>
+<wire x1="29" y1="12" x2="29" y2="9" width="0" layer="19" extent="1-1"/>
+<wire x1="27" y1="14" x2="29" y2="12" width="0" layer="19" extent="1-1"/>
+<wire x1="27" y1="16" x2="27" y2="14" width="0" layer="19" extent="1-1"/>
+<wire x1="24" y1="16" x2="27" y2="16" width="0" layer="19" extent="1-1"/>
+<wire x1="24" y1="14" x2="24" y2="16" width="0" layer="19" extent="1-1"/>
+<wire x1="31" y1="16" x2="27" y2="16" width="0" layer="19" extent="1-1"/>
+<wire x1="33" y1="18" x2="31" y2="16" width="0" layer="19" extent="1-1"/>
+<wire x1="35" y1="20" x2="33" y2="18" width="0" layer="19" extent="1-1"/>
+<wire x1="35" y1="23" x2="35" y2="20" width="0" layer="19" extent="1-1"/>
+<wire x1="35" y1="26" x2="35" y2="23" width="0" layer="19" extent="1-1"/>
+<wire x1="35" y1="29" x2="35" y2="26" width="0" layer="19" extent="1-1"/>
+<wire x1="36" y1="32" x2="35" y2="29" width="0" layer="19" extent="1-1"/>
+<wire x1="36" y1="35" x2="36" y2="32" width="0" layer="19" extent="1-1"/>
+<wire x1="36" y1="38" x2="36" y2="35" width="0" layer="19" extent="1-1"/>
+<wire x1="36" y1="41" x2="36" y2="38" width="0" layer="19" extent="1-1"/>
+<wire x1="33" y1="41" x2="36" y2="41" width="0" layer="19" extent="1-1"/>
+<wire x1="33" y1="38" x2="36" y2="38" width="0" layer="19" extent="1-1"/>
+<wire x1="33" y1="35" x2="36" y2="35" width="0" layer="19" extent="1-1"/>
+<wire x1="33" y1="32" x2="36" y2="32" width="0" layer="19" extent="1-1"/>
+<wire x1="34" y1="44" x2="33" y2="41" width="0" layer="19" extent="1-1"/>
+<wire x1="33" y1="47" x2="34" y2="44" width="0" layer="19" extent="1-1"/>
+<wire x1="36" y1="47" x2="33" y2="47" width="0" layer="19" extent="1-1"/>
+<wire x1="36" y1="50" x2="36" y2="47" width="0" layer="19" extent="1-1"/>
+<wire x1="33" y1="50" x2="33" y2="47" width="0" layer="19" extent="1-1"/>
+<wire x1="30" y1="50" x2="33" y2="50" width="0" layer="19" extent="1-1"/>
+<wire x1="27" y1="50" x2="30" y2="50" width="0" layer="19" extent="1-1"/>
+<wire x1="24" y1="50" x2="27" y2="50" width="0" layer="19" extent="1-1"/>
+<wire x1="39" y1="26" x2="35" y2="26" width="0" layer="19" extent="1-1"/>
+<wire x1="39" y1="23" x2="39" y2="26" width="0" layer="19" extent="1-1"/>
+<wire x1="39" y1="20" x2="39" y2="23" width="0" layer="19" extent="1-1"/>
+<wire x1="39" y1="18" x2="39" y2="20" width="0" layer="19" extent="1-1"/>
+<wire x1="39" y1="15" x2="39" y2="18" width="0" layer="19" extent="1-1"/>
+<wire x1="39" y1="12" x2="39" y2="15" width="0" layer="19" extent="1-1"/>
+<wire x1="37" y1="11" x2="39" y2="12" width="0" layer="19" extent="1-1"/>
+<wire x1="39" y1="9" x2="37" y2="11" width="0" layer="19" extent="1-1"/>
+<wire x1="39" y1="6" x2="39" y2="9" width="0" layer="19" extent="1-1"/>
+<wire x1="39" y1="56" x2="36" y2="50" width="0" layer="19" extent="1-1"/>
+<wire x1="39" y1="59" x2="39" y2="56" width="0" layer="19" extent="1-1"/>
+<wire x1="36" y1="59" x2="39" y2="59" width="0" layer="19" extent="1-1"/>
+<wire x1="33" y1="59" x2="36" y2="59" width="0" layer="19" extent="1-1"/>
+<wire x1="30" y1="59" x2="33" y2="59" width="0" layer="19" extent="1-1"/>
+<wire x1="27" y1="59" x2="30" y2="59" width="0" layer="19" extent="1-1"/>
 <wire x1="28.5" y1="-38.694" x2="18.19" y2="-16.27" width="0" layer="19" extent="1-1"/>
 <wire x1="32" y1="-39.05" x2="28.5" y2="-38.694" width="0" layer="19" extent="1-1"/>
@@
 <signal name="LED-FLOOR">
 <contactref element="CN1" pad="6"/>
+<contactref element="TP4" pad="TP"/>
+<wire x1="23.27" y1="-13.73" x2="35.56" y2="-64.77" width="0" layer="19" extent="1-1"/>
 </signal>
 <signal name="MIRROR">
@@
 <signal name="SIG-FLOOR">
 <contactref element="CN1" pad="5"/>
+<contactref element="TP3" pad="TP"/>
+<wire x1="23.27" y1="-16.27" x2="36.83" y2="-64.77" width="0" layer="19" extent="1-1"/>
 </signal>
 <signal name="SERVO-SIG">
@@
 <contactref element="R10" pad="2"/>
 <contactref element="R9" pad="2"/>
+<contactref element="TP1" pad="TP"/>
+<wire x1="-41.94" y1="-66.985" x2="39.37" y2="-64.77" width="0" layer="19" extent="1-1"/>
 <wire x1="-27.55" y1="-41.306" x2="-41.94" y2="-66.985" width="0" layer="19" extent="1-1"/>
 <wire x1="-15" y1="-41" x2="-27.55" y2="-41.306" width="0" layer="19" extent="1-1"/>

Commit message: ホゲェ
Routing:
- net GND: track 206.7 -> 401.8 mm, vias 48 -> 82
- net +3V3: track 0.00 -> 186.3 mm, vias 0 -> 3
- net SDA: track 0.00 -> 109.0 mm
- net SCL: track 0.00 -> 102.1 mm, vias 0 -> 3
- net LOADCELL-R: track 0.00 -> 67.3 mm, vias 0 -> 2
- net MIRROR: track 0.00 -> 63.2 mm
- net VDD: track 234.2 -> 296.3 mm
- net LED-FLOOR: track 0.00 -> 59.8 mm
- net SIG-FLOOR: track 0.00 -> 54.1 mm, vias 0 -> 4
- net LOADCELL-L: track 0.00 -> 38.9 mm, vias 0 -> 2
- net XSHUT1: track 0.00 -> 29.2 mm
- net XSHUT2: track 0.00 -> 25.0 mm, vias 0 -> 1
- net N$2: track 0.00 -> 17.9 mm
- net N$5: track 0.00 -> 12.9 mm
- net N$1: track 0.00 -> 11.7 mm
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