File: PCB/04-bottom/04-bottom.sch (EAGLE design)
At the start: 28 parts, among them CN1 ML8-R, J1 5267-3, J2 5267-3, J3 5267-3, J4 5267-3, J5 22057045, J6 22057045, J7 5267-3

Commit message: にゅーぷるあっぷ
Parts:
- added R10, R9: 10k, rcl:R-EU_R0402
Connections:
- net +3V3: now also R10.2, R9.2
- net SCL: now also R10.1
- net SDA: now also R9.1
Other:
- note added: "PULL PULL PULL-UP♪ PULL PULL PULL PULL PULL PULL PULL PULL PULL PULL PULL-UP PULL-UP♪"
- note added: "くれらっぷの歌"
- note added: "にゅーぷるあっぷ♪"
Changed lines of the file:
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@@
 <part name="VDD9" library="supply1" library_urn="urn:adsk.eagle:library:371" deviceset="VDD" device=""/>
 <part name="GND18" library="supply1" library_urn="urn:adsk.eagle:library:371" deviceset="GND" device=""/>
+<part name="R9" library="rcl" library_urn="urn:adsk.eagle:library:334" deviceset="R-EU_" device="R0402" package3d_urn="urn:adsk.eagle:package:23547/3" value="10k"/>
+<part name="R10" library="rcl" library_urn="urn:adsk.eagle:library:334" deviceset="R-EU_" device="R0402" package3d_urn="urn:adsk.eagle:package:23547/3" value="10k"/>
+<part name="+3V8" library="supply1" library_urn="urn:adsk.eagle:library:371" deviceset="+3V3" device=""/>
 </parts>
 <sheets>
@@
 <wire x1="0" y1="142.24" x2="162.56" y2="142.24" width="0.1524" layer="94"/>
 <wire x1="93.98" y1="101.6" x2="93.98" y2="0" width="0.1524" layer="94"/>
+<text x="45.72" y="104.14" size="6.4516" layer="94">にゅーぷるあっぷ♪</text>
+<text x="2.54" y="104.14" size="1.778" layer="94">PULL PULL PULL-UP♪
+PULL PULL PULL PULL
+PULL PULL PULL PULL PULL PULL
+PULL-UP PULL-UP♪</text>
+<text x="129.54" y="104.14" size="2.54" layer="94">くれらっぷの歌</text>
+<wire x1="129.54" y1="105.41" x2="154.94" y2="105.41" width="0.1524" layer="94"/>
 </plain>
 <instances>
@@
 <instance part="GND18" gate="1" x="236.22" y="104.14" smashed="yes">
 <attribute name="VALUE" x="233.68" y="101.6" size="1.778" layer="96"/>
+</instance>
+<instance part="R9" gate="G$1" x="86.36" y="132.08" smashed="yes">
+<attribute name="NAME" x="82.55" y="133.5786" size="1.778" layer="95"/>
+<attribute name="VALUE" x="82.55" y="128.778" size="1.778" layer="96"/>
+</instance>
+<instance part="R10" gate="G$1" x="86.36" y="121.92" smashed="yes">
+<attribute name="NAME" x="82.55" y="123.4186" size="1.778" layer="95"/>
+<attribute name="VALUE" x="82.55" y="118.618" size="1.778" layer="96"/>
+</instance>
+<instance part="+3V8" gate="G$1" x="99.06" y="137.16" smashed="yes">
+<attribute name="VALUE" x="101.6" y="134.62" size="1.778" layer="96"/>
 </instance>
 </instances>
@@
 <pinref part="+3V7" gate="G$1" pin="+3V3"/>
 </segment>
+<segment>
+<pinref part="R10" gate="G$1" pin="2"/>
+<wire x1="91.44" y1="121.92" x2="99.06" y2="121.92" width="0.1524" layer="91"/>
+<wire x1="99.06" y1="121.92" x2="99.06" y2="132.08" width="0.1524" layer="91"/>
+<pinref part="R9" gate="G$1" pin="2"/>
+<wire x1="99.06" y1="132.08" x2="99.06" y2="134.62" width="0.1524" layer="91"/>
+<wire x1="91.44" y1="132.08" x2="99.06" y2="132.08" width="0.1524" layer="91"/>
+<junction x="99.06" y="132.08"/>
+<pinref part="+3V8" gate="G$1" pin="+3V3"/>
+</segment>
 </net>
 <net name="SCL" class="0">
@@
 <label x="167.64" y="58.42" size="1.778" layer="95"/>
 </segment>
+<segment>
+<pinref part="R10" gate="G$1" pin="1"/>
+<wire x1="68.58" y1="121.92" x2="81.28" y2="121.92" width="0.1524" layer="91"/>
+<label x="60.96" y="121.92" size="1.778" layer="95"/>
+</segment>
 </net>
 <net name="SDA" class="0">
@@
 <wire x1="187.96" y1="62.23" x2="180.34" y2="62.23" width="0.1524" layer="91"/>
 <label x="167.64" y="62.23" size="1.778" layer="95"/>
+</segment>
+<segment>
+<pinref part="R9" gate="G$1" pin="1"/>
+<wire x1="81.28" y1="132.08" x2="68.58" y2="132.08" width="0.1524" layer="91"/>
+<label x="60.96" y="132.08" size="1.778" layer="95"/>
 </segment>
 </net>
@@
 </drawing>
 <compatibility>
+<note version="6.3" minversion="6.2.2" severity="warning">
+Since Version 6.2.2 text objects can contain more than one line,
+which will not be processed correctly with this version.
+</note>
 <note version="8.2" severity="warning">
 Since Version 8.2, EAGLE supports online libraries. The ids

Commit message: 今度こそ配置完了？
Parts:
- added TP1, TP3, TP4: PTR1TP10R, testpad:PTR1TP10R
- added TP2: PTR1TP10SQ, testpad:PTR1TP10SQ
Connections:
- net +3V3: now also TP1.TP
- net GND: now also TP2.TP
- net LED-FLOOR: now also TP4.TP
- net SIG-FLOOR: now also TP3.TP
Other:
- note added: "FLOOR"
- moved on the sheet: JP1, JP2, JP3, JP4
